File: ATTINY85/BATSENSE2/attiny_batsense2.brd (EAGLE design)
At the start: 45.7 x 37.5 mm, 14 parts

Commit message: final attiny_batsense2 layout
Parts:
- moved R2 15.1 mm to (33.7, 31.8), turned to 270 degrees
- moved R1 5.75 mm to (19.7, 22.9), turned to 0 degrees
Routing:
- net P3: track 4.82 -> 29.7 mm, vias 0 -> 2
- net P4: track 3.18 -> 19.2 mm
- net DGND: track 39.6 -> 24.3 mm, vias 6 -> 4
- net P2: track 0.00 -> 14.5 mm
- net P5: track 0.00 -> 8.50 mm
- net P1: track 0.00 -> 3.04 mm, vias 0 -> 1
- net P0: track 0.00 -> 3.04 mm, vias 0 -> 1
- net +5V: track 97.1 -> 96.6 mm
Changed lines of the file:
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@@
 <setting verticaltext="up"/>
 </settings>
-<grid distance="50" unitdist="mil" unit="mil" style="lines" multiple="1" display="yes" altdistance="0.025" altunitdist="inch" altunit="mil"/>
+<grid distance="25" unitdist="mil" unit="mil" style="lines" multiple="1" display="yes" altdistance="0.025" altunitdist="inch" altunit="mil"/>
 <layers>
 <layer number="1" name="Top" color="4" fill="1" visible="yes" active="yes"/>
@@
 <element name="JP5" library="pinhead" library_urn="urn:adsk.eagle:library:325" package="1X03" package3d_urn="urn:adsk.eagle:package:22458/2" value="" x="41.1688" y="19.4872" rot="R270"/>
 <element name="JP7" library="pinhead" library_urn="urn:adsk.eagle:library:325" package="1X06" package3d_urn="urn:adsk.eagle:package:22472/2" value="" x="32.2768" y="27.1244"/>
-<element name="R1" library="rcl" package="R0805" value="10k" x="25.4" y="22.225" rot="MR270"/>
+<element name="R1" library="rcl" package="R0805" value="10k" x="19.685" y="22.86" rot="MR0"/>
 <element name="C1" library="rcl" package="C1210" value="" x="9.525" y="17.145" rot="MR0"/>
 <element name="C3" library="rcl" package="C1210" value="" x="17.145" y="11.43" rot="MR0"/>
 <element name="JP1" library="pinhead" library_urn="urn:adsk.eagle:library:325" package="1X04" package3d_urn="urn:adsk.eagle:package:22407/2" value="" x="24.2824" y="32.766"/>
-<element name="R2" library="rcl" package="R0805" value="10k" x="20.32" y="24.765" rot="MR180"/>
+<element name="R2" library="rcl" package="R0805" value="10k" x="33.655" y="31.75" rot="MR270"/>
 <element name="JP2" library="pinhead" library_urn="urn:adsk.eagle:library:325" package="1X03" package3d_urn="urn:adsk.eagle:package:22458/2" value="" x="10.8898" y="25.1936" rot="R180"/>
 <element name="LED1" library="led" library_urn="urn:adsk.eagle:library:259" package="LED3MM" package3d_urn="urn:adsk.eagle:package:15797/1" value="" x="10.16" y="31.75" rot="R180"/>
@@
 <vertex x="45.085" y="0"/>
 </polygon>
+<wire x1="8.3498" y1="25.1936" x2="8.3498" y2="28.4802" width="0.8128" layer="16"/>
+<wire x1="8.3498" y1="28.4802" x2="7.62" y2="29.21" width="0.8128" layer="16"/>
+<via x="7.62" y="29.21" extent="1-16" drill="0.8"/>
+<wire x1="7.62" y1="29.21" x2="5.08" y2="29.21" width="0.8128" layer="1"/>
+<wire x1="5.08" y1="29.21" x2="2.54" y2="26.67" width="0.8128" layer="1"/>
+<via x="2.54" y="26.67" extent="1-16" drill="0.8"/>
 <wire x1="41.1688" y1="19.4872" x2="38.5372" y2="19.4872" width="0.8128" layer="16"/>
 <wire x1="38.5372" y1="19.4872" x2="38.1" y2="19.05" width="0.8128" layer="16"/>
-<via x="38.1" y="19.05" extent="1-16" drill="0.35"/>
-<wire x1="38.1" y1="19.05" x2="33.02" y2="19.05" width="0.8128" layer="1"/>
-<wire x1="33.02" y1="19.05" x2="29.21" y2="15.24" width="0.8128" layer="1"/>
-<via x="29.21" y="15.24" extent="1-16" drill="0.35"/>
-<wire x1="8.3498" y1="25.1936" x2="8.3498" y2="28.4802" width="0.8128" layer="16"/>
-<wire x1="8.3498" y1="28.4802" x2="7.62" y2="29.21" width="0.8128" layer="16"/>
-<via x="7.62" y="29.21" extent="1-16" drill="0.35"/>
-<wire x1="7.62" y1="29.21" x2="5.08" y2="29.21" width="0.8128" layer="1"/>
-<wire x1="5.08" y1="29.21" x2="2.54" y2="26.67" width="0.8128" layer="1"/>
-<via x="2.54" y="26.67" extent="1-16" drill="0.35"/>
-<wire x1="20.4724" y1="32.766" x2="20.4724" y2="29.0576" width="0.8128" layer="16"/>
-<wire x1="20.4724" y1="29.0576" x2="21.59" y2="27.94" width="0.8128" layer="16"/>
-<via x="21.59" y="27.94" extent="1-16" drill="0.35"/>
-<wire x1="21.59" y1="27.94" x2="21.59" y2="17.78" width="0.8128" layer="1"/>
-<via x="21.59" y="17.78" extent="1-16" drill="0.35"/>
+<via x="38.1" y="19.05" extent="1-16" drill="0.8"/>
+<wire x1="38.1" y1="19.05" x2="35.56" y2="19.05" width="0.8128" layer="1"/>
+<wire x1="35.56" y1="19.05" x2="29.845" y2="13.335" width="0.8128" layer="1"/>
+<via x="29.845" y="13.335" extent="1-16" drill="0.8"/>
 </signal>
 <signal name="+5V">
@@
 <wire x1="39.37" y1="31.75" x2="39.37" y2="34.29" width="0.8128" layer="16"/>
 <wire x1="39.37" y1="34.29" x2="38.1" y2="35.56" width="0.8128" layer="16"/>
-<wire x1="38.1" y1="35.56" x2="30.8864" y2="35.56" width="0.8128" layer="16"/>
+<wire x1="34.29" y1="35.56" x2="38.1" y2="35.56" width="0.8128" layer="16"/>
+<wire x1="34.29" y1="35.56" x2="30.8864" y2="35.56" width="0.8128" layer="16"/>
 <wire x1="10.795" y1="25.0988" x2="10.8898" y2="25.1936" width="0.8128" layer="16"/>
 <wire x1="10.925" y1="21.59" x2="10.925" y2="17.145" width="0.8128" layer="16"/>
@@
 <wire x1="28.0924" y1="32.766" x2="28.0924" y2="34.1376" width="0.8128" layer="16"/>
 <wire x1="28.0924" y1="34.1376" x2="26.67" y2="35.56" width="0.8128" layer="16"/>
-<wire x1="26.67" y1="35.56" x2="19.05" y2="35.56" width="0.8128" layer="16"/>
-<wire x1="19.05" y1="35.56" x2="17.78" y2="34.29" width="0.8128" layer="16"/>
-<wire x1="17.78" y1="34.29" x2="17.78" y2="26.355" width="0.8128" layer="16"/>
-<wire x1="17.78" y1="26.355" x2="19.37" y2="24.765" width="0.8128" layer="16"/>
-<wire x1="19.05" y1="35.56" x2="8.89" y2="35.56" width="0.8128" layer="16"/>
+<wire x1="26.67" y1="35.56" x2="8.89" y2="35.56" width="0.8128" layer="16"/>
 <wire x1="5.08" y1="31.75" x2="5.08" y2="22.86" width="0.8128" layer="16"/>
 <wire x1="5.08" y1="22.86" x2="6.35" y2="21.59" width="0.8128" layer="16"/>
 <wire x1="6.35" y1="21.59" x2="10.925" y2="21.59" width="0.8128" layer="16"/>
 <wire x1="8.89" y1="35.56" x2="5.08" y2="31.75" width="0.8128" layer="16"/>
-<wire x1="19.37" y1="24.765" x2="25.4" y2="21.275" width="0" layer="19" extent="16-16"/>
+<wire x1="33.655" y1="32.7" x2="33.655" y2="34.925" width="0.8128" layer="16"/>
+<wire x1="33.655" y1="34.925" x2="34.29" y2="35.56" width="0.8128" layer="16"/>
+<wire x1="18.735" y1="22.86" x2="16.51" y2="22.86" width="0.8128" layer="16"/>
+<wire x1="16.51" y1="22.86" x2="15.24" y2="21.59" width="0.8128" layer="16"/>
+<wire x1="15.24" y1="21.59" x2="10.925" y2="21.59" width="0.8128" layer="16"/>
 </signal>
 <signal name="P5">
 <contactref element="JP7" pad="1"/>
 <contactref element="R1" pad="1"/>
-<wire x1="25.4" y1="23.175" x2="25.9268" y2="27.1244" width="0" layer="19" extent="16-16"/>
+<wire x1="20.635" y1="22.86" x2="24.13" y2="22.86" width="0.8128" layer="16"/>
+<wire x1="24.13" y1="22.86" x2="25.4" y2="24.13" width="0.8128" layer="16"/>
+<wire x1="25.4" y1="24.13" x2="25.4" y2="26.5976" width="0.8128" layer="16"/>
+<wire x1="25.4" y1="26.5976" x2="25.9268" y2="27.1244" width="0.8128" layer="16"/>
 </signal>
 <signal name="P4">
@@
 <contactref element="R4" pad="2"/>
 <contactref element="R5" pad="1"/>
-<wire x1="34.925" y1="13.65" x2="34.925" y2="16.83" width="0.8128" layer="16"/>
-<wire x1="34.925" y1="16.83" x2="28.4668" y2="27.1244" width="0" layer="19" extent="16-16"/>
+<wire x1="34.925" y1="16.83" x2="34.925" y2="13.65" width="0.8128" layer="16"/>
+<wire x1="28.4668" y1="27.1244" x2="28.4668" y2="18.5232" width="0.8128" layer="16"/>
+<wire x1="28.4668" y1="18.5232" x2="30.48" y2="16.51" width="0.8128" layer="16"/>
+<wire x1="30.48" y1="16.51" x2="34.605" y2="16.51" width="0.8128" layer="16"/>
+<wire x1="34.605" y1="16.51" x2="34.925" y2="16.83" width="0.8128" layer="16"/>
 </signal>
 <signal name="P3">
@@
 <contactref element="R3" pad="1"/>
 <wire x1="14.605" y1="29.53" x2="14.605" y2="26.3688" width="0.8128" layer="16"/>
-<wire x1="14.605" y1="26.3688" x2="13.4298" y2="25.1936" width="0.8128" layer="16"/>
-<wire x1="14.605" y1="26.3688" x2="31.0068" y2="27.1244" width="0" layer="19" extent="16-16"/>
+<wire x1="13.8031" y1="25.5669" x2="14.605" y2="26.3688" width="0.8128" layer="16"/>
+<wire x1="13.8031" y1="25.5669" x2="13.4298" y2="25.1936" width="0.8128" layer="16"/>
+<wire x1="31.0068" y1="27.1244" x2="31.0068" y2="21.6982" width="0.8128" layer="16"/>
+<wire x1="31.0068" y1="21.6982" x2="31.115" y2="21.59" width="0.8128" layer="16"/>
+<via x="31.115" y="21.59" extent="1-16" drill="0.8"/>
+<wire x1="31.115" y1="21.59" x2="24.765" y2="21.59" width="0.8128" layer="1"/>
+<wire x1="24.765" y1="21.59" x2="20.955" y2="25.4" width="0.8128" layer="1"/>
+<wire x1="20.955" y1="25.4" x2="18.415" y2="25.4" width="0.8128" layer="1"/>
+<wire x1="18.415" y1="25.4" x2="17.78" y2="26.035" width="0.8128" layer="1"/>
+<via x="17.78" y="26.035" extent="1-16" drill="0.8"/>
+<wire x1="17.78" y1="26.035" x2="14.2712" y2="26.035" width="0.8128" layer="16"/>
+<wire x1="14.2712" y1="26.035" x2="13.8031" y2="25.5669" width="0.8128" layer="16"/>
 </signal>
 <signal name="P2">
@@
 <contactref element="R2" pad="2"/>
 <contactref element="JP1" pad="3"/>
-<wire x1="25.5524" y1="32.766" x2="33.5468" y2="27.1244" width="0" layer="19" extent="1-1"/>
-<wire x1="21.27" y1="24.765" x2="25.5524" y2="32.766" width="0" layer="19" extent="16-16"/>
+<wire x1="33.5468" y1="27.1244" x2="33.5468" y2="30.6918" width="0.8128" layer="16"/>
+<wire x1="33.5468" y1="30.6918" x2="33.655" y2="30.8" width="0.8128" layer="16"/>
+<wire x1="33.5468" y1="30.6918" x2="30.6918" y2="30.6918" width="0.8128" layer="16"/>
+<wire x1="30.6918" y1="30.6918" x2="29.845" y2="29.845" width="0.8128" layer="16"/>
+<wire x1="29.845" y1="29.845" x2="26.67" y2="29.845" width="0.8128" layer="16"/>
+<wire x1="26.67" y1="29.845" x2="25.4" y2="31.115" width="0.8128" layer="16"/>
+<wire x1="25.4" y1="31.115" x2="25.4" y2="32.6136" width="0.8128" layer="16"/>
+<wire x1="25.4" y1="32.6136" x2="25.5524" y2="32.766" width="0.8128" layer="16"/>
 </signal>
 <signal name="P1">
 <contactref element="JP7" pad="5"/>
+<via x="36.195" y="24.13" extent="1-16" drill="0.8" diameter="1.3"/>
+<wire x1="36.0868" y1="27.1244" x2="36.0868" y2="24.2382" width="0.8128" layer="16"/>
+<wire x1="36.0868" y1="24.2382" x2="36.195" y2="24.13" width="0.8128" layer="16"/>
 </signal>
 <signal name="P0">
 <contactref element="JP7" pad="6"/>
+<via x="38.735" y="24.13" extent="1-16" drill="0.8" diameter="1.3"/>
+<wire x1="38.6268" y1="27.1244" x2="38.6268" y2="24.2382" width="0.8128" layer="16"/>
+<wire x1="38.6268" y1="24.2382" x2="38.735" y2="24.13" width="0.8128" layer="16"/>
 </signal>
 <signal name="NA">
