File: WIRINGS/multi_sense/multi_sense.sch (EAGLE design)
At the start: 8 parts

Commit message: pinout documentation
Other:
- note added: "RST - A0 - TEMT Sig D0 - D5 - PIR Sig D6 - (relay one) D7 - DHT PWR D8 - TEMT PWR 3.3V - PIR PWR"
- note added: "WEMOS Pinning: Tx - Rx - D1 - Neo Sig D2 - D3 - DHT Sig D4 - G - NEO GND, PIR GND, TEMPT GND, DHT GND 5V - NEO PWR"
- note removed: "WEMOS Pinning: Tx - RST - Rx - A0 - TEMT Sig D1 - Neo Sig D0 - D2 - D5 - PIR Sig D3 - DHT Sig D6 - D4 - D7 - DHT PWR G - GND D8 - TEMT PWR 5V - NEO PWR 3.3V - PIR PWR GND - NEO GND, PIR GND, TEMPT GND, DHT GND"
Changed lines of the file:
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@@
 <setting verticaltext="up"/>
 </settings>
-<grid distance="50" unitdist="mil" unit="mil" style="lines" multiple="1" display="no" altdistance="0.01" altunitdist="inch" altunit="inch"/>
+<grid distance="0.1" unitdist="inch" unit="inch" style="lines" multiple="1" display="no" altdistance="0.01" altunitdist="inch" altunit="inch"/>
 <layers>
 <layer number="1" name="Top" color="4" fill="1" visible="no" active="no"/>
@@
 <plain>
 <text x="-22.86" y="255.27" size="1.778" layer="91">WEMOS Pinning:
-Tx -                    RST -
-Rx -                    A0 - TEMT Sig
-D1 - Neo Sig       D0 -
-D2 -                    D5 - PIR Sig
-D3 - DHT Sig       D6 -
-D4 -                    D7 - DHT PWR
-G -   GND            D8 - TEMT PWR
-5V - NEO PWR     3.3V - PIR PWR
-GND - NEO GND, PIR GND, TEMPT GND, DHT GND</text>
+Tx -
+Rx -
+D1 - Neo Sig
+D2 -
+D3 - DHT Sig
+D4 -
+G -   NEO GND, PIR GND, TEMPT GND, DHT GND
+5V - NEO PWR </text>
+<text x="38.1" y="255.27" size="1.778" layer="91">
+RST -
+A0 - TEMT Sig
+D0 -
+D5 - PIR Sig
+D6 - (relay one)
+D7 - DHT PWR
+D8 - TEMT PWR
+3.3V - PIR PWR</text>
 </plain>
 <instances>
