File: WEMOS/WEMOS_GPIO/wemos_gpio.sch (EAGLE design)
At the start: 16 parts, among them IC1 MCP23017SP, IC2 ULN2801A

Commit message: reworked structure
Parts:
- added C3, C4: (no value), rcl:CPOL-EUTT5D7
- added C5, C6: (no value), rcl:C-EUC1210
Connections:
- net +3V3: now also C3.+, C5.1
- net +5V: now also C4.+, C6.1
- net DGND: now also C3.-, C4.-, C5.2, C6.2
Changed lines of the file:
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@@
 <part name="JP5" library="pinhead" library_urn="urn:adsk.eagle:library:325" deviceset="PINHD-1X3" device="" package3d_urn="urn:adsk.eagle:package:22458/2"/>
 <part name="SUPPLY3" library="supply2" library_urn="urn:adsk.eagle:library:372" deviceset="DGND" device=""/>
+<part name="C3" library="rcl" library_urn="urn:adsk.eagle:library:334" deviceset="CPOL-EU" device="TT5D7" package3d_urn="urn:adsk.eagle:package:23314/1"/>
+<part name="C4" library="rcl" library_urn="urn:adsk.eagle:library:334" deviceset="CPOL-EU" device="TT5D7" package3d_urn="urn:adsk.eagle:package:23314/1"/>
+<part name="C5" library="rcl" deviceset="C-EU" device="C1210"/>
+<part name="C6" library="rcl" deviceset="C-EU" device="C1210"/>
+<part name="+3V1" library="supply1" deviceset="+3V3" device=""/>
+<part name="P+2" library="supply1" library_urn="urn:adsk.eagle:library:371" deviceset="+5V" device=""/>
+<part name="SUPPLY4" library="supply2" library_urn="urn:adsk.eagle:library:372" deviceset="DGND" device=""/>
+<part name="SUPPLY6" library="supply2" library_urn="urn:adsk.eagle:library:372" deviceset="DGND" device=""/>
 </parts>
 <sheets>
@@
 <instance part="JP5" gate="A" x="-91.44" y="157.48" rot="MR0"/>
 <instance part="SUPPLY3" gate="G$1" x="-69.85" y="142.24"/>
+<instance part="C3" gate="G$1" x="-96.52" y="266.7"/>
+<instance part="C4" gate="G$1" x="-71.12" y="266.7"/>
+<instance part="C5" gate="G$1" x="-88.9" y="266.7"/>
+<instance part="C6" gate="G$1" x="-63.5" y="266.7"/>
+<instance part="+3V1" gate="G$1" x="-96.52" y="279.4"/>
+<instance part="P+2" gate="1" x="-71.12" y="278.13"/>
+<instance part="SUPPLY4" gate="G$1" x="-96.52" y="252.73"/>
+<instance part="SUPPLY6" gate="G$1" x="-71.12" y="252.73"/>
 </instances>
 <busses>
@@
 <wire x1="-25.4" y1="144.78" x2="-35.56" y2="144.78" width="0.1524" layer="91"/>
 <label x="-34.29" y="144.78" size="1.778" layer="95"/>
+</segment>
+<segment>
+<pinref part="+3V1" gate="G$1" pin="+3V3"/>
+<pinref part="C3" gate="G$1" pin="+"/>
+<wire x1="-96.52" y1="276.86" x2="-96.52" y2="274.32" width="0.1524" layer="91"/>
+<pinref part="C5" gate="G$1" pin="1"/>
+<wire x1="-96.52" y1="274.32" x2="-96.52" y2="269.24" width="0.1524" layer="91"/>
+<wire x1="-96.52" y1="274.32" x2="-88.9" y2="274.32" width="0.1524" layer="91"/>
+<wire x1="-88.9" y1="274.32" x2="-88.9" y2="269.24" width="0.1524" layer="91"/>
+<junction x="-96.52" y="274.32"/>
 </segment>
 </net>
@@
 <label x="-83.82" y="200.66" size="1.778" layer="95"/>
 </segment>
+<segment>
+<pinref part="C3" gate="G$1" pin="-"/>
+<pinref part="SUPPLY4" gate="G$1" pin="DGND"/>
+<wire x1="-96.52" y1="261.62" x2="-96.52" y2="257.81" width="0.1524" layer="91"/>
+<pinref part="C5" gate="G$1" pin="2"/>
+<wire x1="-96.52" y1="257.81" x2="-96.52" y2="255.27" width="0.1524" layer="91"/>
+<wire x1="-88.9" y1="261.62" x2="-88.9" y2="257.81" width="0.1524" layer="91"/>
+<wire x1="-88.9" y1="257.81" x2="-96.52" y2="257.81" width="0.1524" layer="91"/>
+<junction x="-96.52" y="257.81"/>
+</segment>
+<segment>
+<pinref part="C4" gate="G$1" pin="-"/>
+<pinref part="SUPPLY6" gate="G$1" pin="DGND"/>
+<wire x1="-71.12" y1="261.62" x2="-71.12" y2="256.54" width="0.1524" layer="91"/>
+<pinref part="C6" gate="G$1" pin="2"/>
+<wire x1="-71.12" y1="256.54" x2="-71.12" y2="255.27" width="0.1524" layer="91"/>
+<wire x1="-63.5" y1="261.62" x2="-63.5" y2="256.54" width="0.1524" layer="91"/>
+<wire x1="-63.5" y1="256.54" x2="-71.12" y2="256.54" width="0.1524" layer="91"/>
+<junction x="-71.12" y="256.54"/>
+</segment>
 </net>
 <net name="GPB0" class="0">
@@
 <label x="-83.82" y="193.04" size="1.778" layer="95"/>
 </segment>
-</net>
+<segment>
+<pinref part="P+2" gate="1" pin="+5V"/>
+<pinref part="C4" gate="G$1" pin="+"/>
+<wire x1="-71.12" y1="275.59" x2="-71.12" y2="273.05" width="0.1524" layer="91"/>
+<pinref part="C6" gate="G$1" pin="1"/>
+<wire x1="-71.12" y1="273.05" x2="-71.12" y2="269.24" width="0.1524" layer="91"/>
+<wire x1="-71.12" y1="273.05" x2="-63.5" y2="273.05" width="0.1524" layer="91"/>
+<wire x1="-63.5" y1="273.05" x2="-63.5" y2="269.24" width="0.1524" layer="91"/>
+<junction x="-71.12" y="273.05"/>
+</segment>
+</net>
