File: WEMOS/WEMOS_GPIO/wemos_gpio_7x.brd (EAGLE design)
At the start: 45.7 x 62.2 mm, 24 parts

Commit message: reworked wemos gpio, reworked wiring for garden control
Parts:
- removed DHT, DHT1: (no value), pinhead:1X03
- removed JP1: (no value), jumper:JP4Q
- removed MCP_DOWN, MCP_LEFT, MCP_RIGHT, ULN_IN, ULN_OUT, WEMOS_LEFT, WEMOS_RIGHT: (no value), pinhead:1X08
- removed MCP_UP: (no value), pinhead:1X10
- removed POWER1, RELAY_1_1, RELAY_2_1, WEMOS_USB: (no value), pinhead:1X02
- removed RELAY_1, RELAY_2: (no value), pinhead:1X06
- removed ULN_PWR: (no value), pinhead:1X04
- added C1, C2: (no value), rcl:C1210
- added IC1: MCP23017SP, SWI_COMMONS:DIL28-3
- added IC2: ULN2801A, uln-udn:DIL18
- added JP2: (no value), pinhead:1X10
- added JP3, JP4: (no value), pinhead:1X08
- added JP5: (no value), pinhead:1X03
- added U$1: TEMP-HUM-SENSOR-DHT22, SWI_COMMONS:TEMP-HUM-SENSOR-DHT22
- added WEMOS1: (no value), SWI_COMMONS:WEMOS-D1-MINI
- R1, R5: device rcl:0207/10 -> rcl@1:M1206
- R2, R3, R4: value (none) -> 10k; device rcl:0204/7 -> rcl@1:M1206
- moved R5 374.1 mm to (76.3, 63.5), flipped to the bottom, turned to 180 degrees
- moved R4 339.1 mm to (45.7, 60.3), flipped to the bottom, turned to 180 degrees
- moved R3 321.1 mm to (48.2, 54.6), flipped to the bottom
- moved R2 303.2 mm to (50.7, 48.9), flipped to the bottom
- moved R1 179.1 mm to (53.3, 43.2), flipped to the bottom
- moved U$2 31.1 mm to (42.4, 1.91)
Connections:
- removed net DHT_GND: DHT.3, DHT1.3
- removed net DHT_VCC: DHT.1, DHT1.1
- removed net GND_1: JP1.2, JP1.4, POWER1.2
- removed net INTA: MCP_DOWN.8
- removed net INTB: MCP_DOWN.7
- removed net N$1: R2.1
- removed net N$11: JP1.5
- removed net N$12: JP1.1
- removed net N$13: ULN_OUT.1
- removed net N$14: ULN_OUT.2
- removed net N$15: ULN_OUT.3
- removed net N$16: ULN_OUT.4
- removed net N$17: ULN_OUT.5
- removed net N$18: ULN_OUT.6
- removed net N$19: ULN_OUT.7
- removed net N$20: ULN_OUT.8
- removed net N$21: R5.2
- removed net N$23: ULN_IN.1
- removed net N$24: ULN_IN.2
- removed net N$25: ULN_IN.3
- removed net N$26: ULN_IN.4
- removed net N$27: ULN_IN.5
- removed net N$28: ULN_IN.6
- removed net N$29: ULN_IN.7
- removed net N$30: ULN_IN.8
- removed net N$31: R5.1
- removed net N$32: R3.1, R4.1
- removed net N$33: R3.2
- removed net N$4: R1.2
- removed net N$49: ULN_PWR.1
- removed net N$5: R1.1
- removed net N$50: ULN_PWR.2
- removed net N$51: ULN_PWR.3
- removed net N$52: ULN_PWR.4
- removed net N$8: JP1.7
- removed net N$9: JP1.3
- removed net POWER_5V_1: JP1.6, JP1.8, POWER1.1
- removed net R1_GND: RELAY_1.6
- removed net R1_J_VCC: RELAY_1_1.1
- removed net R1_R1: RELAY_1.2
- removed net R1_R2: RELAY_1.3
- removed net R1_R3: RELAY_1.4
- removed net R1_R4: RELAY_1.5
- removed net R1_VCC: RELAY_1.1, RELAY_1_1.2
- removed net R2_GND: RELAY_2.6
- removed net R2_J_VCC: RELAY_2_1.1
- removed net R2_R1: RELAY_2.2
- removed net R2_R2: RELAY_2.3
- removed net R2_R4: RELAY_2.4, RELAY_2.5
- removed net R2_VCC: RELAY_2.1, RELAY_2_1.2
- removed net SCA: MCP_DOWN.4
- removed net W_3_3V: WEMOS_LEFT.1
- removed net W_5V: WEMOS_RIGHT.1
- removed net W_A0: WEMOS_LEFT.7
- removed net W_D0: WEMOS_LEFT.6
- removed net W_D1_SCL: WEMOS_RIGHT.6
- removed net W_D2_SDA: WEMOS_RIGHT.5
- removed net W_D3: WEMOS_RIGHT.4
- removed net W_D4: WEMOS_RIGHT.3
- removed net W_D5: WEMOS_LEFT.5
- removed net W_D6: WEMOS_LEFT.4
- removed net W_D7: WEMOS_LEFT.3
- removed net W_D8: WEMOS_LEFT.2
- removed net W_GND: WEMOS_RIGHT.2
- removed net W_RESET: WEMOS_LEFT.8
- removed net W_RX: WEMOS_RIGHT.7
- removed net W_TX: WEMOS_RIGHT.8
- new net 5V: WEMOS1.5V
- new net A0: IC1.15, R1.2
- new net A1: IC1.16, R2.2
- new net A2: IC1.17, R3.2
- new net ANALOG: WEMOS1.A0
- new net D0: WEMOS1.D0
- new net D4: WEMOS1.D4
- new net D5: WEMOS1.D5
- new net DHTE_DATA: JP5.2, WEMOS1.D8
- new net DHTE_PWR: JP5.1, WEMOS1.D6
- new net DHT_PWR: R5.2, U$1.1, WEMOS1.D7
- new net N$3: U$1.3
- new net PGPA0: IC2.11, JP3.8
- new net PGPA1: IC2.12, JP3.7
- new net PGPA2: IC2.13, JP3.6
- new net PGPA3: IC2.14, JP3.5
- new net PGPA4: IC2.15, JP3.4
- new net PGPA5: IC2.16, JP3.3
- new net PGPA6: IC2.17, JP3.2
- new net PGPA7: IC2.18, JP3.1
- new net RESET: WEMOS1.RESET
- new net RX: WEMOS1.RX
- new net SDA: IC1.13, WEMOS1.D2
- net +3V3: now also C1.1, IC1.9, JP2.1, JP2.2, JP2.3, JP2.4, R4.2, WEMOS1.3V3; no longer MCP_DOWN.1, MCP_UP.1, MCP_UP.2, MCP_UP.3
- net +5V: now also C2.1, IC2.10, JP2.10, JP2.8, JP2.9; no longer MCP_UP.5, MCP_UP.6, WEMOS_USB.2
- net DGND: now also C1.2, C2.2, IC1.10, IC2.9, JP2.5, JP2.6, JP2.7, JP5.3, R1.1, R2.1, R3.1, U$1.4, WEMOS1.GND; no longer MCP_DOWN.2, MCP_DOWN.5, MCP_UP.10, MCP_UP.8, MCP_UP.9, WEMOS_USB.1
- net DHT_DATA: now also R5.1, U$1.2, WEMOS1.D3; no longer DHT.2, DHT1.2
- net GPA0: now also IC1.21, IC2.8; no longer MCP_RIGHT.1
- net GPA1: now also IC1.22, IC2.7; no longer MCP_RIGHT.2
- net GPA2: now also IC1.23, IC2.6; no longer MCP_RIGHT.3
- net GPA3: now also IC1.24, IC2.5; no longer MCP_RIGHT.4
- net GPA4: now also IC1.25, IC2.4; no longer MCP_RIGHT.5
- net GPA5: now also IC1.26, IC2.3; no longer MCP_RIGHT.6
- net GPA6: now also IC1.27, IC2.2; no longer MCP_RIGHT.7
- net GPA7: now also IC1.28, IC2.1; no longer MCP_RIGHT.8
- net GPB0: now also IC1.1, JP4.1; no longer MCP_LEFT.1
- net GPB1: now also IC1.2, JP4.2; no longer MCP_LEFT.2
- net GPB2: now also IC1.3, JP4.3; no longer MCP_LEFT.3
- net GPB3: now also IC1.4, JP4.4; no longer MCP_LEFT.4
- net GPB4: now also IC1.5, JP4.5; no longer MCP_LEFT.5
- net GPB5: now also IC1.6, JP4.6; no longer MCP_LEFT.6
- net GPB6: now also IC1.7, JP4.7; no longer MCP_LEFT.7
- net GPB7: now also IC1.8, JP4.8; no longer MCP_LEFT.8
- net NRES: now also IC1.18, R4.1; no longer MCP_DOWN.6
- net SCL: now also IC1.12, WEMOS1.D1; no longer MCP_DOWN.3
Routing:
- net +3V3: track 66.6 -> 220.5 mm
- net +5V: track 2.54 -> 66.1 mm
- net DHT_PWR: track 0.00 -> 48.2 mm
- net DGND: track 0.00 -> 46.8 mm, vias 0 -> 4
- net SDA: track 0.00 -> 43.3 mm
- net DHT_DATA: track 0.00 -> 38.7 mm
- net INTA: track 31.9 -> 0.00 mm
- net INTB: track 30.2 -> 0.00 mm
- net A2: track 0.00 -> 21.4 mm
- net SCL: track 19.3 -> 37.6 mm
- net SCA: track 16.2 -> 0.00 mm
- net A1: track 0.00 -> 15.7 mm
- net DHTE_PWR: track 0.00 -> 10.8 mm
- net A0: track 0.00 -> 9.98 mm
- net DHTE_DATA: track 0.00 -> 9.57 mm
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Other:
- board size 45.7 x 62.2 mm -> 92.7 x 70.2 mm
- board text added: "PN39024R1B1"
- board text added: "WSHIELD_WEMOS_GPIO"
- board text removed: "PN39022R1B1"
- board text removed: "WSHIELD_MCP_BASIC"

Commit message: reworked structure
Parts:
- added C3, C4: (no value), rcl@1:TT5D7
- added C5, C6: (no value), rcl:C1210
- moved U$2 34.7 mm to (8.13, 7.53)
- moved JP4 2.00 mm to (27.7, 14.5)
- moved C1 2.00 mm to (47.6, 17.1)
- moved C2 2.00 mm to (40.6, 41.2)
- moved IC1 2.00 mm to (35.3, 27.4)
- moved IC2 2.00 mm to (26.4, 41.1)
- moved JP2 2.00 mm to (6.99, 32.9)
- moved JP3 2.00 mm to (25.2, 53.9)
- moved JP5 2.00 mm to (82.5, 13.2)
- moved R1 2.00 mm to (53.3, 41.2)
- moved R2 2.00 mm to (50.7, 46.9)
- moved R3 2.00 mm to (48.2, 52.6)
- moved R4 2.00 mm to (45.7, 58.3)
- moved R5 2.00 mm to (76.3, 61.5)
- moved U$1 2.00 mm to (73.7, 57.7)
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Connections:
- net +3V3: now also C3.+, C5.1
- net +5V: now also C4.+, C6.1
- net DGND: now also C3.-, C4.-, C5.2, C6.2
Routing:
- net +5V: track 66.1 -> 69.6 mm
- net +3V3: track 220.5 -> 223.7 mm
Other:
- board size 92.7 x 70.2 mm -> 92.7 x 68.2 mm
