File: WEMOS/WEMOS_SENSE/wemos_sense.brd (EAGLE design)
At the start: 52.7 x 93.2 mm, 27 parts, among them IC1 MCP23017SP

Commit message: updated wemos and diverse boards
Parts:
- removed C3: (no value), rcl:C1210
- removed JP10, JP8: (no value), pinhead:1X04
- removed JP6: (no value), pinhead:1X02
- removed JP7: (no value), jumper:JP2
- removed S1, S2: (no value), switch-omron:B3F-10XX
- added D4: 1N4148DO35-7, diode:DO35-7
- added JP6-TEMT6000, NEOPIX: (no value), pinhead:1X03
- added LED4: (no value), led:CHIP-LED0805
- added R40, R41, R9: (no value), rcl:R0805
- added R8: 10k, rcl:R0805
- added T5: BC547, transistor:TO92
- added X2, X9: (no value), con-wago-508:W237-132
- JP2: device pinhead:1X04 -> pinhead:1X02
- U$4: value MOTION-PIR-DYP-ME003 -> RELAYPTH; device diy-modules:MOTION-PIR-DYP-ME003 -> SRD-05VDC-SL-C:SRD-05VDC-SL-C
- moved JP2 364.9 mm to (-61.0, -328.9), turned to 0 degrees
- moved U$4 295.2 mm to (-54.6, -290.8)
- renumbered JP4 to JP4-OLED, JP5 to JP5-PIRAM312, JP9 to JP9-BME280
Connections:
- removed net GND: U$3.4, U$4.1
- removed net VCC: U$4.3
- removed net VDD: U$3.1
- new net N$22: D4.A, T5.3, U$4.COIL0
- new net N$24: U$4.SWCOMMON, X9.1
- new net N$25: U$4.SWOPEN, X2.2
- new net N$26: U$4.SWCLOSED, X9.2
- new net N$27: R40.2, T5.2
- new net N$31: LED4.A, R9.1
- net +3V3: now also JP5-PIRAM312.1
- net +5V: now also D4.C, NEOPIX.1, U$4.COIL1
- net A0: now also JP6-TEMT6000.1
- net D3: now also R8.2, U$3.2
- net D4: now also NEOPIX.2
- net D5/SCK: now also JP5-PIRAM312.2, JP6-TEMT6000.2
- net D6/MISO: now also R40.1, R41.1, R9.2
- net D7/MOSI: now also R8.1, U$3.1
- net D8/SS: now also JP6-TEMT6000.3
- net DGND: now also JP5-PIRAM312.3, LED4.C, NEOPIX.3, R41.2, T5.1, U$3.4
- net RX: now also JP2.2
- net TX: now also JP2.1

Commit message: layout started
Parts:
- removed C4: (no value), rcl:C1210
- removed JP1: (no value), pinhead:1X07
- removed LED4: (no value), led:CHIP-LED0805
- removed R9: (no value), rcl:R0805
- added JP3, JP4: (no value), pinhead:1X08
- added LED1: (no value), led:LED3MM
- added R42: (no value), rcl:R0805
- moved R40 407.8 mm to (47.0, 77.5), flipped to the bottom, turned to 270 degrees
- moved T5 405.7 mm to (36.8, 74.9), turned to 270 degrees
- moved D4 402.9 mm to (31.8, 80.0), turned to 270 degrees
- moved R41 394.3 mm to (36.8, 67.3), flipped to the bottom, turned to 90 degrees
- moved X2 391.3 mm to (5.08, 82.5), turned to 90 degrees
- moved X9 379.5 mm to (5.08, 72.4), turned to 90 degrees
- moved U$4 378.1 mm to (19.1, 80.0)
- moved JP2 363.2 mm to (43.2, 19.1), turned to 270 degrees
- moved R7 315.7 mm to (44.5, 62.2), flipped to the bottom, turned to 270 degrees
- moved R5 304.7 mm to (47.0, 62.2), flipped to the bottom, turned to 270 degrees
- moved NEOPIX 304.6 mm to (45.7, 5.08), turned to 90 degrees
- moved R6 303.8 mm to (44.5, 55.9), flipped to the bottom, turned to 270 degrees
- moved R3 293.9 mm to (49.5, 62.2), flipped to the bottom, turned to 270 degrees
- moved R4 292.9 mm to (47.0, 55.9), flipped to the bottom, turned to 270 degrees
- moved JP6-TEMT6000 288.3 mm to (6.35, 12.7), turned to 270 degrees
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Connections:
- removed net N$24: U$4.SWCOMMON, X9.1
- removed net N$26: U$4.SWCLOSED, X9.2
- removed net N$31: LED4.A, R9.1
- new net N$1: IC1.21, JP3.1
- new net N$10: IC1.2, JP4.2
- new net N$11: IC1.3, JP4.3
- new net N$12: IC1.4, JP4.4
- new net N$13: IC1.5, JP4.5
- new net N$14: IC1.6, JP4.6
- new net N$15: IC1.7, JP4.7
- new net N$16: IC1.8, JP4.8
- new net N$17: U$4.SWCOMMON, X9.2
- new net N$18: U$4.SWCLOSED, X9.1
- new net N$19: LED1.A, R42.1
- new net N$2: IC1.22, JP3.2
- new net N$3: IC1.23, JP3.3
- new net N$4: IC1.24, JP3.4
- new net N$5: IC1.25, JP3.5
- new net N$6: IC1.26, JP3.6
- new net N$7: IC1.27, JP3.7
- new net N$8: IC1.28, JP3.8
- new net N$9: IC1.1, JP4.1
- net +3V3: no longer JP1.7
- net +5V: no longer JP1.5
- net D4: now also NEOPIX.3; no longer NEOPIX.2
- net D5/SCK: no longer JP1.1
- net D6/MISO: now also R42.2; no longer JP1.2, R9.2
- net D7/MOSI: no longer JP1.3
- net D8/SS: no longer JP1.4
- net DGND: now also LED1.K, NEOPIX.2; no longer JP1.6, LED4.C, NEOPIX.3

Commit message: shematic ready, started placing
Parts:
- moved LED1 15.3 mm to (41.9, 85.1), turned to 180 degrees
Routing:
- net N$25: track 0.00 -> 23.8 mm
- net N$18: track 0.00 -> 22.7 mm
- net N$22: track 0.00 -> 22.2 mm
- net +5V: track 0.00 -> 21.1 mm
- net N$17: track 0.00 -> 8.63 mm
Changed lines of the file:
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@@
 <attribute name="VALUE" x="15.24" y="31.115" size="1.27" layer="27"/>
 </element>
-<element name="LED1" library="led" library_urn="urn:adsk.eagle:library:259" package="LED3MM" package3d_urn="urn:adsk.eagle:package:15797/1" value="" x="43.18" y="69.85" smashed="yes" rot="R90">
-<attribute name="NAME" x="41.275" y="66.421" size="1.27" layer="25" ratio="10"/>
-<attribute name="POPULARITY" value="97" x="43.18" y="69.85" size="1.778" layer="27" rot="R90" display="off"/>
-<attribute name="VALUE" x="44.831" y="71.755" size="1.27" layer="27" ratio="10" rot="R90"/>
+<element name="LED1" library="led" library_urn="urn:adsk.eagle:library:259" package="LED3MM" package3d_urn="urn:adsk.eagle:package:15797/1" value="" x="41.91" y="85.09" smashed="yes" rot="R180">
+<attribute name="NAME" x="45.339" y="83.185" size="1.27" layer="25" ratio="10" rot="R90"/>
+<attribute name="POPULARITY" value="97" x="41.91" y="85.09" size="1.778" layer="27" rot="R180" display="off"/>
+<attribute name="VALUE" x="40.005" y="86.741" size="1.27" layer="27" ratio="10" rot="R180"/>
 </element>
 </elements>
@@
 <contactref element="U$4" pad="COIL1"/>
 <contactref element="D4" pad="C"/>
-<wire x1="13.66" y1="85.89" x2="31.75" y2="83.82" width="0" layer="19" extent="1-1"/>
+<wire x1="13.66" y1="85.89" x2="18.27" y2="81.28" width="0.3048" layer="1"/>
+<wire x1="18.27" y1="81.28" x2="29.21" y2="81.28" width="0.3048" layer="1"/>
+<wire x1="29.21" y1="81.28" x2="31.75" y2="83.82" width="0.3048" layer="1"/>
 <wire x1="38.1" y1="2.54" x2="31.75" y2="83.82" width="0" layer="19" extent="1-1"/>
 <wire x1="45.72" y1="2.54" x2="38.1" y2="2.54" width="0" layer="19" extent="1-1"/>
@@
 <contactref element="WEMOS1" pad="A0"/>
 <contactref element="JP6-TEMT6000" pad="1"/>
-<wire x1="49.53" y1="54.93" x2="49.53" y2="61.28" width="0" layer="19" extent="16-16"/>
+<wire x1="49.53" y1="61.28" x2="49.53" y2="54.93" width="0" layer="19" extent="16-16"/>
 <wire x1="49.53" y1="49.53" x2="49.53" y2="54.93" width="0" layer="19" extent="16-16"/>
 <wire x1="15.24" y1="17.78" x2="49.53" y2="49.53" width="0" layer="19" extent="1-1"/>
@@
 <contactref element="R7" pad="2"/>
 <contactref element="IC1" pad="17"/>
-<wire x1="44.45" y1="56.83" x2="44.45" y2="61.28" width="0" layer="19" extent="16-16"/>
+<wire x1="44.45" y1="61.28" x2="44.45" y2="56.83" width="0" layer="19" extent="16-16"/>
 <wire x1="44.45" y1="49.53" x2="44.45" y2="56.83" width="0" layer="19" extent="16-16"/>
 </signal>
@@
 <contactref element="LED1" pad="K"/>
 <contactref element="NEOPIX" pad="2"/>
-<wire x1="36.83" y1="73.66" x2="43.18" y2="71.12" width="0" layer="19" extent="1-1"/>
+<wire x1="36.83" y1="73.66" x2="40.64" y2="85.09" width="0" layer="19" extent="1-1"/>
 <wire x1="36.83" y1="68.26" x2="36.83" y2="73.66" width="0" layer="19" extent="16-16"/>
-<wire x1="44.45" y1="63.18" x2="43.18" y2="71.12" width="0" layer="19" extent="16-16"/>
+<wire x1="44.45" y1="63.18" x2="40.64" y2="85.09" width="0" layer="19" extent="16-16"/>
 <wire x1="46.99" y1="63.18" x2="44.45" y2="63.18" width="0" layer="19" extent="16-16"/>
 <wire x1="49.53" y1="63.18" x2="46.99" y2="63.18" width="0" layer="19" extent="16-16"/>
@@
 <contactref element="D4" pad="A"/>
 <contactref element="T5" pad="3"/>
+<wire x1="13.66" y1="73.89" x2="19.78" y2="80.01" width="0.3048" layer="1"/>
+<wire x1="27.94" y1="80.01" x2="31.75" y2="76.2" width="0.3048" layer="1"/>
+<wire x1="19.78" y1="80.01" x2="27.94" y2="80.01" width="0.3048" layer="1"/>
 <wire x1="31.75" y1="76.2" x2="36.83" y2="76.2" width="0" layer="19" extent="1-1"/>
-<wire x1="13.66" y1="73.89" x2="31.75" y2="76.2" width="0" layer="19" extent="1-1"/>
 </signal>
 <signal name="N$25">
 <contactref element="U$4" pad="SWOPEN"/>
 <contactref element="X2" pad="2"/>
-<wire x1="5.715" y1="85.09" x2="25.66" y2="85.89" width="0" layer="19" extent="1-1"/>
+<wire x1="25.66" y1="85.89" x2="21.38" y2="90.17" width="2.54" layer="16"/>
+<wire x1="10.795" y1="90.17" x2="5.715" y2="85.09" width="2.54" layer="16"/>
+<wire x1="21.38" y1="90.17" x2="10.795" y2="90.17" width="2.54" layer="16"/>
 </signal>
 <signal name="N$27">
@@
 <contactref element="X9" pad="2"/>
 <contactref element="U$4" pad="SWCOMMON"/>
-<wire x1="5.715" y1="74.93" x2="11.66" y2="79.89" width="0" layer="19" extent="1-1"/>
+<wire x1="11.66" y1="79.89" x2="6.7" y2="74.93" width="2.54" layer="16"/>
+<wire x1="6.7" y1="74.93" x2="5.08" y2="74.93" width="2.54" layer="16"/>
+<wire x1="5.08" y1="74.93" x2="5.715" y2="74.93" width="0" layer="19" extent="16-16"/>
 </signal>
 <signal name="N$18">
 <contactref element="X9" pad="1"/>
 <contactref element="U$4" pad="SWCLOSED"/>
-<wire x1="5.715" y1="69.85" x2="25.66" y2="73.89" width="0" layer="19" extent="1-1"/>
+<wire x1="25.66" y1="73.89" x2="20.35" y2="68.58" width="2.54" layer="16"/>
+<wire x1="6.985" y1="68.58" x2="5.715" y2="69.85" width="2.54" layer="16"/>
+<wire x1="20.35" y1="68.58" x2="6.985" y2="68.58" width="2.54" layer="16"/>
 </signal>
 <signal name="N$19">
 <contactref element="R42" pad="1"/>
 <contactref element="LED1" pad="A"/>
-<wire x1="43.18" y1="68.58" x2="43.18" y2="76.52" width="0" layer="19" extent="16-16"/>
+<wire x1="43.18" y1="85.09" x2="43.18" y2="76.52" width="0" layer="19" extent="16-16"/>
 </signal>
 </signals>

Commit message: layout progress update
Parts:
- moved R8 22.6 mm to (26.7, 17.8), turned to 90 degrees
- moved R41 12.5 mm to (48.3, 72.4), turned to 270 degrees
- moved C1 5.24 mm to (26.7, 5.08)
- moved R42 5.24 mm to (48.3, 78.7), turned to 270 degrees
- moved C2 5.08 mm to (26.7, 11.4)
- moved R40 4.02 mm to (43.2, 76.2)
- moved LED1 1.27 mm to (43.2, 85.1)
Routing:
- net D7/MOSI: track 0.00 -> 56.2 mm
- net D3: track 0.00 -> 55.6 mm
- net +3V3: track 0.00 -> 36.8 mm
- net SCA: track 0.00 -> 18.3 mm
- net SCL: track 0.00 -> 18.3 mm
- net D8/SS: track 0.00 -> 11.0 mm
- net A0: track 0.00 -> 9.94 mm
- net D6/MISO: track 0.00 -> 9.80 mm
- net D5/SCK: track 0.00 -> 8.89 mm
- net N$9: track 0.00 -> 7.62 mm
- net N$16: track 0.00 -> 7.62 mm
- net N$15: track 0.00 -> 7.62 mm
- net N$14: track 0.00 -> 7.62 mm
- net N$13: track 0.00 -> 7.62 mm
- net N$12: track 0.00 -> 7.62 mm
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- added copper zone on layer 16, net DGND
