File: WEMOS/WEMOS_SENSE/wemos_sense.sch (EAGLE design)
At the start: 27 parts, among them IC1 MCP23017SP

Commit message: updated wemos and diverse boards
Parts:
- removed C3: (no value), rcl:C-EUC1210
- removed JP10, JP8: (no value), pinhead:PINHD-1X4
- removed JP5: (no value), pinhead:PINHD-1X3
- removed JP6: (no value), pinhead:PINHD-1X2
- removed JP7: (no value), jumper:JP2E
- removed S1, S2: (no value), switch-omron:10-XX
- added D4: 1N4148DO35-7, diode:1N4148DO35-7
- added JP5-PIRAM312, JP6-TEMT6000, NEOPIX: (no value), pinhead:PINHD-1X3
- added LED4: (no value), led:LEDCHIP-LED0805
- added R40, R41, R9: (no value), rcl:R-EU_R0805
- added R8: 10k, rcl:R-EU_R0805
- added T5: BC547, transistor:BC547
- added X2, X9: (no value), con-wago-508:W237-02P
- JP2: device pinhead:PINHD-1X4 -> pinhead:PINHD-1X2
- U$4: value MOTION-PIR-DYP-ME003 -> RELAYPTH; device diy-modules:MOTION-PIR-DYP-ME003 -> SRD-05VDC-SL-C:RELAYPTH
- renumbered JP4 to JP4-OLED, JP9 to JP9-BME280
Connections:
- new net N$22: D4.A, T5.C, U$4.COIL0
- new net N$24: U$4.SWCOMMON, X9-1.KL
- new net N$25: U$4.SWOPEN, X2-2.KL
- new net N$26: U$4.SWCLOSE, X9-2.KL
- new net N$27: R40.2, T5.B
- new net N$31: LED4.A, R9.1
- net +3V3: now also JP5-PIRAM312.1
- net +5V: now also D4.C, NEOPIX.1, U$4.COIL1
- net A0: now also JP6-TEMT6000.1
- net D3: now also R8.2, U$3.DAT
- net D4: now also NEOPIX.2
- net D5/SCK: now also JP5-PIRAM312.2, JP6-TEMT6000.2
- net D6/MISO: now also R40.1, R41.1, R9.2
- net D7/MOSI: now also R8.1, U$3.VDD
- net D8/SS: now also JP6-TEMT6000.3
- net DGND: now also JP5-PIRAM312.3, LED4.C, NEOPIX.3, R41.2, T5.E, U$3.GND
- net RX: now also JP2.2
- net TX: now also JP2.1
Other:
- note added: "WEMOS Pinning: Tx - RST - Rx - A0 - TEMT Sig D1 - D0 - D2 - NEO Sig D5 - PIR Sig D3 - DHT Sig D6 - D4 - D7 - DHT PWR G - D8 - TEMT PWR 5V - NEO pwr 3.3V - PIR PWR"
- note removed: "BME280"
- note removed: "OLED"
- moved on the sheet: C4, U$3

Commit message: layout started
Parts:
- removed C4: (no value), rcl:C-EUC1210
- removed JP1: (no value), pinhead:PINHD-1X7
- removed LED4: (no value), led:LEDCHIP-LED0805
- added JP3, JP4: (no value), pinhead:PINHD-1X8
- added LED1: (no value), led:LED3MM
- renumbered R9 to R42
Connections:
- removed net N$24: U$4.SWCOMMON, X9-1.KL
- removed net N$26: U$4.SWCLOSE, X9-2.KL
- removed net N$31: LED4.A, R42.1
- new net N$1: IC1.GPA0, JP3.1
- new net N$10: IC1.GPB1, JP4.2
- new net N$11: IC1.GPB2, JP4.3
- new net N$12: IC1.GPB3, JP4.4
- new net N$13: IC1.GPB4, JP4.5
- new net N$14: IC1.GPB5, JP4.6
- new net N$15: IC1.GPB6, JP4.7
- new net N$16: IC1.GPB7, JP4.8
- new net N$17: U$4.SWCOMMON, X9-2.KL
- new net N$18: U$4.SWCLOSE, X9-1.KL
- new net N$19: LED1.A, R42.1
- new net N$2: IC1.GPA1, JP3.2
- new net N$3: IC1.GPA2, JP3.3
- new net N$4: IC1.GPA3, JP3.4
- new net N$5: IC1.GPA4, JP3.5
- new net N$6: IC1.GPA5, JP3.6
- new net N$7: IC1.GPA6, JP3.7
- new net N$8: IC1.GPA7, JP3.8
- new net N$9: IC1.GPB0, JP4.1
- net +3V3: no longer JP1.7
- net +5V: no longer JP1.5
- net D4: now also NEOPIX.3; no longer NEOPIX.2
- net D5/SCK: no longer JP1.1
- net D6/MISO: no longer JP1.2
- net D7/MOSI: no longer JP1.3
- net D8/SS: no longer JP1.4
- net DGND: now also LED1.C, NEOPIX.2; no longer JP1.6, LED4.C, NEOPIX.3
